File: minifrank.kicad_pcb (KiCad board)
At the start: 2 copper layers, 54 x 58 mm, 70 parts, among them J1 Conn_01x02, U1 NCP1117-3.3_SOT223, U2 W25Q128JVS, U3 RP2040, Y1 ABM8-272-T3

Commit message: HW Rev 1.0
Parts:
- added L1: LED, LED_SMD:LED_0805_2012Metric_Pad1.15x1.40mm_HandSolder, F.Cu at (123.6, 64.4)
- added L2: LED, LED_SMD:LED_0805_2012Metric_Pad1.15x1.40mm_HandSolder, F.Cu at (115.4, 58.0)
- added R27: 10K, Resistor_SMD:R_0805_2012Metric_Pad1.20x1.40mm_HandSolder, F.Cu at (103.2, 43.4)
- added R28: 10K, Resistor_SMD:R_0805_2012Metric_Pad1.20x1.40mm_HandSolder, F.Cu at (101.6, 40.4)
- added R29: 10K, Resistor_SMD:R_0805_2012Metric_Pad1.20x1.40mm_HandSolder, F.Cu at (101.6, 38.2)
- added R30: 10K, Resistor_SMD:R_0805_2012Metric_Pad1.20x1.40mm_HandSolder, F.Cu at (102.0, 30.4)
- added R31: 1K, Resistor_SMD:R_0805_2012Metric_Pad1.20x1.40mm_HandSolder, F.Cu at (119.4, 58.0)
- added R32: 1K, Resistor_SMD:R_0805_2012Metric_Pad1.20x1.40mm_HandSolder, F.Cu at (90.4, 62.5)
- added SW1: Reset Button, LIBS:Button_SMD_6x6x5, F.Cu at (146.9, 37.2)
- DB1: renamed from DB4; footprint LIBS:DSUB-9_Male_EdgeMount_P2.77mm -> Connector_Dsub:DSUB-9_Male_EdgeMount_P2.77mm
- J1: footprint Connector_PinHeader_2.54mm:PinHeader_1x02_P2.54mm_Vertical -> LIBS:Boot_Jumper
- moved G*** 21.6 mm to (91.2, 34.6), turned to -90 degrees
- moved Y1 2.44 mm to (118.5, 53.4)
- moved C18 2.21 mm to (130.2, 45.8)
- moved C14 2.20 mm to (130.2, 48.0)
- moved C1 2.20 mm to (114.4, 53.6)
- moved C19 1.40 mm to (132.4, 41.8)
- moved C9 1.40 mm to (136.6, 41.8)
- moved C4 0.82 mm to (133.6, 28.0)
- moved C6 0.70 mm to (131.4, 28.0)
- moved D3 0.50 mm to (109.2, 55.9)
- moved D2 0.40 mm to (111.6, 55.9)
- renumbered C22 to C1, C24 to C10, C6 to C11, C14 to C12, C7 to C13, C8 to C14, C9 to C15, C10 to C16, C16 to C17, C11 to C18, C12 to C19, C23 to C2, C3 to C20, C17 to C21, C20 to C22, C18 to C23, C21 to C24, C15 to C3, C19 to C4, C4 to C5, C1 to C6, C5 to C7, C13 to C8, C2 to C9, D6 to D1, D1 to D2, D2 to D3, R14 to R1, R12 to R10, R23 to R11, R24 to R12, R5 to R13, R9 to R14, R16 to R15, R20 to R16, R3 to R17, R6 to R18, R7 to R19, R58 to R2, R11 to R20, R4 to R21, R8 to R22, R15 to R23, R17 to R24, R18 to R25, R19 to R26, R13 to R3, R21 to R4, R1 to R5, R2 to R6, R22 to R7, R25 to R8, R10 to R9, U2 to U1, U1 to U2
Routing:
- net Net-(L1-A): track 0.00 -> 39.0 mm, vias 0 -> 2
- net +3V3: track 203.6 -> 238.2 mm, vias 4 -> 7
- net /GPIO25: track 0.00 -> 31.9 mm, vias 0 -> 2
- net /GPIO5: track 25.6 -> 46.1 mm, vias 2 -> 4
- net VBUS: track 203.5 -> 223.7 mm, vias 3 -> 5
- net /RUN: track 0.00 -> 19.9 mm, vias 0 -> 2
- net /GPIO2: track 26.0 -> 42.6 mm, vias 2 -> 3
- net /GPIO4: track 32.1 -> 46.8 mm
- net /GPIO3: track 25.6 -> 33.3 mm, vias 2 -> 4
- net /GPIO26: track 41.8 -> 46.6 mm
- net Net-(C2-Pad1): track 5.60 -> 8.61 mm, vias 0 -> 2
- net /GPIO14: track 23.5 -> 26.2 mm
- net /XIN: track 13.7 -> 11.7 mm
- net Net-(L2-A): track 0.00 -> 2.00 mm
- net /GPIO15: track 31.7 -> 29.8 mm
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Other:
- board text added: "HW Rev. 1.0"

Commit message: HW Rev. 1.0 (final)
Parts:
- DB1: footprint Connector_Dsub:DSUB-9_Male_EdgeMount_P2.77mm -> LIBS:DSUB-9
- renumbered L2 to L1, L1 to L2, R8 to R10, R9 to R11, R10 to R12, R11 to R13, R12 to R14, R13 to R15, R14 to R16, R15 to R17, R16 to R18, R27 to R19, R28 to R20, R29 to R21, R30 to R22, R17 to R23, R18 to R24, R19 to R25, R20 to R26, R21 to R27, R22 to R28, R23 to R29, R24 to R30, R25 to R31, R26 to R32, R31 to R7, R32 to R8, R7 to R9
Routing:
- net GND: vias 56 -> 59
