File: minifrank.kicad_pcb (KiCad board)
At the start: 2 copper layers, 54 x 58 mm, 79 parts, among them J1 Conn_01x02, SW1 Reset Button, U1 W25Q128JVS, U2 NCP1117-3.3_SOT223, U3 RP2040, Y1 ABM8-272-T3

Commit message: Minor fixes
Parts:
- removed the G*** at (91.2, 34.6)

Commit message: HW Rev 1.1
Parts:
- removed G***: LOGO, LIBS:Mini_Frank_QR
- removed J1: Conn_01x02, LIBS:Boot_Jumper
- removed R3: DNF, Resistor_SMD:R_0805_2012Metric_Pad1.20x1.40mm_HandSolder
- added SW2: Flash Button, LIBS:Button_SMD_3x3x2, F.Cu at (109.0, 26.7)
- DB1: footprint LIBS:DSUB-9 -> Connector_Dsub:DSUB-9_Male_EdgeMount_P2.77mm
- SW1: footprint LIBS:Button_SMD_6x6x5 -> LIBS:Button_SMD_3x3x2
- U2: footprint Package_TO_SOT_SMD:SOT-223-3_TabPin2 -> LIBS:Medved_SOT-223-3_TabPin2
- moved SW1 12.7 mm to (138.6, 46.8), turned to -90 degrees
- moved L2 2.26 mm to (122.0, 62.8)
- moved R1 2.20 mm to (111.6, 31.0)
- moved D1 1.40 mm to (124.0, 60.2)
- moved KB1 0.81 mm to (94.0, 73.8)
Routing:
- net /PS/2 CLK: track 32.2 -> 21.7 mm
- net /PS/2 DATA: track 19.1 -> 10.5 mm
- net +3V3: track 238.2 -> 232.8 mm
- net /RUN: track 19.9 -> 15.3 mm
- net Net-(L2-A): track 39.0 -> 35.6 mm
- net /~{USB_BOOT}: track 3.70 -> 5.70 mm
- net /GPIO3: track 33.3 -> 35.2 mm
- net /GPIO6: track 18.8 -> 17.4 mm
- net /GPIO5: track 46.1 -> 47.1 mm
- net VBUS: track 223.7 -> 222.7 mm
- net /GPIO26: track 46.6 -> 47.5 mm
- net Net-(C22-Pad1): track 49.4 -> 50.1 mm
- net /GPIO27: track 52.0 -> 51.5 mm
- net GND: track 32.2 -> 32.8 mm, vias 59 -> 61
Other:
- board text added: "HW Rev. 1.1"
- board text added: "© 2024 Mikhail Matveev https://rh1.dev"
- board text removed: "HW Rev. 1.0"

Commit message: Minor updates
Parts:
- moved L2 1.26 mm to (123.0, 63.6)
Routing:
- net Net-(L2-A): track 35.6 -> 36.4 mm
Changed lines of the file:
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@@
 			(pintype "passive+no_connect")
 		)
-		(model "${KICAD8_3DMODEL_DIR}/Connector_Dsub.3dshapes/DSUB-9_Male_EdgeMount_P2.77mm.wrl"
+		(model "${KICAD8_3DMODEL_DIR}/Connector_Dsub.3dshapes/DSUB-9_Female_Vertical_P2.77x2.84mm.wrl"
 			(offset
-				(xyz 0 0 0)
+				(xyz 5.5 -3 0.5)
 			)
 			(scale
@@
 			)
 			(rotate
-				(xyz 0 0 0)
+				(xyz -90 0 0)
 			)
 		)
@@
 	(footprint "LED_SMD:LED_0805_2012Metric_Pad1.15x1.40mm_HandSolder"
 		(layer "F.Cu")
-		(at 122.025 62.8)
+		(at 123 63.6)
 		(descr "LED SMD 0805 (2012 Metric), square (rectangular) end terminal, IPC_7351 nominal, (Body size source: https://docs.google.com/spreadsheets/d/1BsfQQcO9C6DZCsRaXUlFlo91Tg2WpOkGARC1WS5S8t0/edit?usp=sharing), generated with kicad-footprint-generator")
 		(tags "LED handsolder")
@@
 		)
 	)
-	(gr_text "HW Rev. 1.1"
-		(at 87.6 49.2 270)
-		(layer "F.SilkS")
-		(effects
-			(font
-				(size 0.8 0.8)
-				(thickness 0.13)
-			)
-			(justify right bottom mirror)
-		)
-	)
 	(segment
 		(start 111.1 76.7)
@@
 	)
 	(via
-		(at 125.69 62.22)
+		(at 125.662591 61.627409)
 		(size 0.6)
 		(drill 0.35)
@@
 	)
 	(segment
-		(start 125.210052 67.35)
-		(end 118.45 67.35)
+		(start 131.225001 55.725001)
+		(end 131.225 55.725002)
 		(width 0.2)
 		(layer "F.Cu")
@@
 	)
 	(segment
-		(start 125.555714 67.004338)
-		(end 125.210052 67.35)
+		(start 124.817818 58.84)
+		(end 124.647818 59.01)
 		(width 0.2)
 		(layer "F.Cu")
@@
 	)
 	(segment
-		(start 126.66065 44.8075)
-		(end 126.56065 44.9075)
+		(start 116.25 69.55)
+		(end 116.25 73.95)
 		(width 0.2)
 		(layer "F.Cu")
@@
 	)
 	(segment
-		(start 128.961534 58.84)
-		(end 124.817818 58.84)
+		(start 125.210052 67.35)
+		(end 118.45 67.35)
 		(width 0.2)
 		(layer "F.Cu")
@@
 	)
 	(segment
-		(start 116.25 69.55)
-		(end 116.25 73.95)
+		(start 126.66065 44.8075)
+		(end 126.56065 44.9075)
 		(width 0.2)
 		(layer "F.Cu")
@@
 	)
 	(segment
-		(start 124.15 62.264034)
-		(end 125.555714 63.669748)
+		(start 125.555714 63.555714)
+		(end 125.555714 67.004338)
 		(width 0.2)
 		(layer "F.Cu")
@@
 	)
 	(segment
-		(start 126.838469 44.8075)
-		(end 126.66065 44.8075)
+		(start 124.39 59.01)
+		(end 124.15 59.25)
 		(width 0.2)
 		(layer "F.Cu")
@@
 	)
 	(segment
-		(start 126.56065 44.9075)
-		(end 126.0975 44.9075)
+		(start 128.961534 58.84)
+		(end 124.817818 58.84)
 		(width 0.2)
 		(layer "F.Cu")
@@
 	)
 	(segment
-		(start 124.15 59.25)
-		(end 124.15 62.264034)
+		(start 126.838469 44.8075)
+		(end 126.66065 44.8075)
 		(width 0.2)
 		(layer "F.Cu")
@@
 	)
 	(segment
-		(start 125.555714 63.669748)
-		(end 125.555714 67.004338)
+		(start 124.15 59.25)
+		(end 124.15 62.15)
 		(width 0.2)
 		(layer "F.Cu")
@@
 	)
 	(segment
-		(start 131.225001 55.725001)
-		(end 131.225 55.725002)
+		(start 126.56065 44.9075)
+		(end 126.0975 44.9075)
 		(width 0.2)
 		(layer "F.Cu")
@@
 	)
 	(segment
-		(start 131.225 56.576534)
-		(end 128.961534 58.84)
+		(start 125.555714 67.004338)
+		(end 125.210052 67.35)
 		(width 0.2)
 		(layer "F.Cu")
@@
 	)
 	(segment
-		(start 127.435105 45.404136)
-		(end 126.838469 44.8075)
+		(start 131.225 56.576534)
+		(end 128.961534 58.84)
 		(width 0.2)
 		(layer "F.Cu")
@@
 	)
 	(segment
-		(start 124.817818 58.84)
-		(end 124.647818 59.01)
+		(start 124.15 62.15)
+		(end 125.555714 63.555714)
 		(width 0.2)
 		(layer "F.Cu")
@@
 	)
 	(segment
-		(start 116.25 73.95)
-		(end 117.1 74.8)
+		(start 127.435105 45.404136)
+		(end 126.838469 44.8075)
 		(width 0.2)
 		(layer "F.Cu")
@@
 	)
 	(segment
-		(start 124.39 59.01)
-		(end 124.15 59.25)
+		(start 116.25 73.95)
+		(end 117.1 74.8)
 		(width 0.2)
 		(layer "F.Cu")
@@
 	)
 	(segment
+		(start 120.95 64.55)
+		(end 123.075 64.55)
+		(width 0.2)
+		(layer "F.Cu")
+		(net 88)
+	)
+	(segment
 		(start 94.7 65.85)
 		(end 95 65.85)
@@
 	)
 	(segment
-		(start 121.45 64.4)
-		(end 123.05 62.8)
+		(start 95 65.85)
+		(end 94.9 65.85)
 		(width 0.2)
 		(layer "F.Cu")
@@
 	)
 	(segment
-		(start 120.8 64.4)
-		(end 121.45 64.4)
+		(start 91.4 62.55)
+		(end 94.7 65.85)
 		(width 0.2)
 		(layer "F.Cu")
@@
 	)
 	(segment
-		(start 95 65.85)
-		(end 94.9 65.85)
+		(start 123.075 64.55)
+		(end 124.025 63.6)
 		(width 0.2)
 		(layer "F.Cu")
@@
 	)
 	(segment
-		(start 91.4 62.55)
-		(end 94.7 65.85)
+		(start 120.8 64.4)
+		(end 120.95 64.55)
 		(width 0.2)
 		(layer "F.Cu")

Commit message: HW Rev. 1.2
Parts:
- U2: footprint LIBS:Medved_SOT-223-3_TabPin2 -> Package_TO_SOT_SMD:SOT-223-3_TabPin2
- moved L1 0.30 mm to (115.7, 58.0)
Connections:
- SW1 pad 2: /RUN -> GND
- SW1 pad 3: GND -> /RUN
- SW2 pad 2: /~{USB_BOOT} -> GND
- SW2 pad 3: GND -> /~{USB_BOOT}
Routing:
- net /~{USB_BOOT}: track 5.70 -> 10.4 mm
- net /RUN: track 15.3 -> 18.1 mm
- net /PS/2 CLK: track 21.7 -> 23.1 mm
Other:
- board text added: "HW Rev. 1.2"
- board text removed: "HW Rev. 1.1"
Changed lines of the file:
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@@
 	(paper "A4")
 	(title_block
-		(title "RP2040 Minimal Design Example")
-		(date "2024-01-16")
-		(rev "1.1")
-		(company "Raspberry Pi Ltd")
+		(title "Mini FRANK")
+		(date "2024-11-13")
+		(rev "1.2")
+		(company "Mikhail Matveev")
+		(comment 1 "https://github.com/xtremespb/minifrank")
 	)
 	(layers
@@
 		(tags "Switch")
 		(property "Reference" "SW2"
-			(at 1.8 1.64 180)
+			(at 1.8 1.64 360)
 			(layer "F.SilkS")
 			(effects
@@
 		)
 		(property "Value" "Flash Button"
-			(at 2.15 1.59 -90)
+			(at 2.15 1.59 90)
 			(layer "F.SilkS")
 			(hide yes)
@@
 		)
 		(property "Footprint" "LIBS:Button_SMD_3x3x2"
-			(at 0 0 -90)
+			(at 0 0 90)
 			(layer "F.Fab")
 			(hide yes)
@@
 		)
 		(property "Datasheet" ""
-			(at 0 0 -90)
+			(at 0 0 90)
 			(layer "F.Fab")
 			(hide yes)
@@
 		)
 		(property "Description" "Push button switch, generic, symbol, four pins"
-			(at 0 0 -90)
+			(at 0 0 90)
 			(layer "F.Fab")
 			(hide yes)
@@
 			(layers "F.Cu" "F.Paste" "F.Mask")
 			(roundrect_rratio 0.1312335958)
-			(net 7 "/~{USB_BOOT}")
+			(net 1 "GND")
 			(pinfunction "2")
 			(pintype "passive")
@@
 			(layers "F.Cu" "F.Paste" "F.Mask")
 			(roundrect_rratio 0.1312335958)
-			(net 1 "GND")
+			(net 7 "/~{USB_BOOT}")
 			(pinfunction "3")
 			(pintype "passive")
@@
 			(layers "F.Cu" "F.Paste" "F.Mask")
 			(roundrect_rratio 0.1312335958)
-			(net 34 "/RUN")
+			(net 1 "GND")
 			(pinfunction "2")
 			(pintype "passive")
@@
 			(layers "F.Cu" "F.Paste" "F.Mask")
 			(roundrect_rratio 0.1312335958)
-			(net 1 "GND")
+			(net 34 "/RUN")
 			(pinfunction "3")
 			(pintype "passive")
@@
 		)
 	)
-	(footprint "LIBS:Medved_SOT-223-3_TabPin2"
+	(footprint "Package_TO_SOT_SMD:SOT-223-3_TabPin2"
 		(layer "F.Cu")
 		(at 134.4 34.8 -90)
@@
 		(tags "CMS SOT")
 		(property "Reference" "U2"
-			(at -4.4 4.6 -90)
+			(at -5 -3.75 0)
 			(layer "F.SilkS")
 			(effects
@@
 			)
 		)
-		(property "Footprint" "LIBS:Medved_SOT-223-3_TabPin2"
+		(property "Footprint" "Package_TO_SOT_SMD:SOT-223-3_TabPin2"
 			(at 0 0 -90)
 			(unlocked yes)
@@
 	(footprint "LED_SMD:LED_0805_2012Metric_Pad1.15x1.40mm_HandSolder"
 		(layer "F.Cu")
-		(at 115.375 58)
+		(at 115.675 58)
 		(descr "LED SMD 0805 (2012 Metric), square (rectangular) end terminal, IPC_7351 nominal, (Body size source: https://docs.google.com/spreadsheets/d/1BsfQQcO9C6DZCsRaXUlFlo91Tg2WpOkGARC1WS5S8t0/edit?usp=sharing), generated with kicad-footprint-generator")
 		(tags "LED handsolder")
@@
 	)
 	(gr_line
-		(start 127.4 61.8)
-		(end 127.4 61.4)
+		(start 127.6 60.4)
+		(end 127.6 60)
 		(stroke
 			(width 0.12)
@@
 	)
 	(gr_line
-		(start 127.6 61.8)
-		(end 127.4 61.8)
+		(start 127.8 60.4)
+		(end 127.6 60.4)
 		(stroke
 			(width 0.12)
@@
 	)
 	(gr_line
-		(start 127.4 61.4)
-		(end 127.6 61.4)
+		(start 127.6 60)
+		(end 127.8 60)
 		(stroke
 			(width 0.12)
@@
 	)
 	(gr_line
-		(start 127.6 61.4)
-		(end 127.6 61.8)
+		(start 127.8 60)
+		(end 127.8 60.4)
 		(stroke
 			(width 0.12)
@@
 	)
 	(gr_line
-		(start 127.5 61.8)
-		(end 127.5 61.4)
+		(start 127.7 60.4)
+		(end 127.7 60)
 		(stroke
 			(width 0.12)
@@
 		(layer "Edge.Cuts")
 	)
-	(gr_text "HW Rev. 1.1"
+	(gr_text "HW Rev. 1.2"
 		(at 86.4 68.8 270)
 		(layer "B.Cu")
@@
 		)
 	)
-	(gr_text "HW Rev. 1.1"
+	(gr_text "HW Rev. 1.2"
 		(at 86.4 68.8 270)
 		(layer "B.SilkS")
@@
 	)
 	(segment
+		(start 137.99 50.6)
+		(end 138.03 50.56)
+		(width 0.2)
+		(layer "F.Cu")
+		(net 1)
+	)
+	(segment
 		(start 125.825 30.81)
 		(end 126.005 30.81)
@@
 	)
 	(segment
-		(start 111 30.6)
-		(end 111.6 30)
-		(width 0.15)
+		(start 106.15 28.15)
+		(end 106.15 26.295)
+		(width 0.2)
 		(layer "F.Cu")
 		(net 7)
 	)
 	(segment
-		(start 106.15 30.6)
-		(end 111 30.6)
-		(width 0.15)
+		(start 111.6 30)
+		(end 110.9 30)
+		(width 0.2)
+		(layer "F.Cu")
+		(net 7)
+	)
+	(segment
+		(start 106.2 28.2)
+		(end 106.15 28.15)
+		(width 0.2)
+		(layer "F.Cu")
+		(net 7)
+	)
+	(segment
+		(start 106.15 28.15)
+		(end 106.15 30.505)
+		(width 0.2)
+		(layer "F.Cu")
+		(net 7)
+	)
+	(segment
+		(start 109.1 28.2)
+		(end 106.2 28.2)
+		(width 0.2)
+		(layer "F.Cu")
+		(net 7)
+	)
+	(segment
+		(start 110.9 30)
+		(end 109.1 28.2)
+		(width 0.2)
 		(layer "F.Cu")
 		(net 7)
@@
 	)
 	(segment
-		(start 104.3 73.9)
-		(end 103.35 72.95)
+		(start 118.659234 44.1075)
+		(end 118.359234 43.8075)
 		(width 0.2)
 		(layer "F.Cu")
@@
 	)
 	(segment
-		(start 118.659234 44.1075)
-		(end 118.359234 43.8075)
+		(start 116.5925 43.8075)
+		(end 116.1 44.3)
 		(width 0.2)
 		(layer "F.Cu")
@@
 	)
 	(segment
-		(start 116.5925 43.8075)
-		(end 116.1 44.3)
+		(start 107.3 55.387)
+		(end 109.2 53.487)
 		(width 0.2)
 		(layer "F.Cu")
@@
 	)
 	(segment
-		(start 107.3 55.387)
-		(end 109.2 53.487)
+		(start 107.3 58.714034)
+		(end 107.3 55.387)
 		(width 0.2)
 		(layer "F.Cu")
@@
 	)
 	(segment
-		(start 103.35 72.95)
-		(end 103.35 62.664034)
+		(start 110.25 42.572182)
+		(end 110.25 42.85)
 		(width 0.2)
 		(layer "F.Cu")
@@
 	)
 	(segment
-		(start 103.35 62.664034)
+		(start 103.2 62.814034)
 		(end 107.3 58.714034)
 		(width 0.2)
@@
 	)
 	(segment
-		(start 107.3 58.714034)
-		(end 107.3 55.387)
+		(start 119.2225 44.1075)
+		(end 118.659234 44.1075)
 		(width 0.2)
 		(layer "F.Cu")
@@
 	)
 	(segment
-		(start 110.25 42.572182)
-		(end 110.25 42.85)
+		(start 110.25 42.85)
+		(end 107.35 45.75)
 		(width 0.2)
 		(layer "F.Cu")
@@
 	)
 	(segment
-		(start 119.2225 44.1075)
-		(end 118.659234 44.1075)
+		(start 104.3 73.9)
+		(end 103.2 72.8)
 		(width 0.2)
 		(layer "F.Cu")
@@
 	)
 	(segment
-		(start 110.25 42.85)
-		(end 107.35 45.75)
+		(start 103.2 72.8)
+		(end 103.2 62.814034)
 		(width 0.2)
 		(layer "F.Cu")
@@
 	)
 	(segment
+		(start 128.81 50.6)
+		(end 133.5 50.6)
+		(width 0.2)
+		(layer "F.Cu")
+		(net 34)
+	)
+	(segment
+		(start 135.775 48.275)
+		(end 135.775 46.35)
+		(width 0.2)
+		(layer "F.Cu")
+		(net 34)
+	)
+	(segment
 		(start 124.2 50.45)
 		(end 124.46 50.19)
@@
 	)
 	(segment
-		(start 128.81 50.6)
-		(end 137.99 50.6)
+		(start 133.5 50.6)
+		(end 135.775 48.325)
 		(width 0.2)
 		(layer "F.Cu")
@@
 	)
 	(segment
-		(start 137.99 50.6)
-		(end 138.03 50.56)
+		(start 135.775 48.325)
+		(end 135.775 50.56)
 		(width 0.2)
 		(layer "F.Cu")
@@
 	(segment
 		(start 99.4 73.35)
-		(end 99.4 72.627818)
+		(end 99.6 73.55)
 		(width 0.2)
 		(layer "F.Cu")
@@
 	)
 	(segment
-		(start 102.3 69.727818)
+		(start 101.45 70.35)
 		(end 102.3 69.5)
 		(width 0.2)
@@
 	)
 	(segment
-		(start 99.4 72.627818)
-		(end 102.3 69.727818)
+		(start 101.45 73.55)
+		(end 101.45 70.35)
+		(width 0.2)
+		(layer "F.Cu")
+		(net 56)
+	)
+	(segment
+		(start 99.6 73.55)
+		(end 101.45 73.55)
 		(width 0.2)
 		(layer "F.Cu")
