File: minifrank.kicad_sch (KiCad schematic)
At the start: 64 parts, among them J1 Conn_01x02, U1 NCP1117-3.3_SOT223, U2 W25Q128JVS, U3 RP2040, Y1 ABM8-272-T3

Commit message: HW Rev 1.0
Parts:
- added L1, L2: LED, LED_SMD:LED_0805_2012Metric_Pad1.15x1.40mm_HandSolder, symbol Device:LED
- added R27, R28, R29, R30: 10K, Resistor_SMD:R_0805_2012Metric_Pad1.20x1.40mm_HandSolder, symbol Device:R
- added R31, R32: 1K, Resistor_SMD:R_0805_2012Metric_Pad1.20x1.40mm_HandSolder, symbol Device:R
- added SW1: Reset Button, LIBS:Button_SMD_6x6x5, symbol Switch:SW_Push_Dual
- renumbered C22 to C1, C24 to C10, C6 to C11, C14 to C12, C7 to C13, C8 to C14, C9 to C15, C10 to C16, C16 to C17, C11 to C18, C12 to C19, C23 to C2, C3 to C20, C17 to C21, C20 to C22, C18 to C23, C21 to C24, C15 to C3, C19 to C4, C4 to C5, C1 to C6, C5 to C7, C13 to C8, C2 to C9, D6 to D1, D1 to D2, D2 to D3, DB4 to DB1, R14 to R1, R12 to R10, R23 to R11, R24 to R12, R5 to R13, R9 to R14, R16 to R15, R20 to R16, R3 to R17, R6 to R18, R7 to R19, R58 to R2, R11 to R20, R4 to R21, R8 to R22, R15 to R23, R17 to R24, R18 to R25, R19 to R26, R13 to R3, R21 to R4, R1 to R5, R2 to R6, R22 to R7, R25 to R8, R10 to R9, U2 to U1, U1 to U2
Connections:
- net +3V3: now also R27.2, R28.2, R29.2, R30.2, R32.2
- net GND: now also L1.1 (K), L2.1 (K), SW1.1, SW1.3
- net GPIO2: now also R27.1
- net GPIO25: now also R31.2
- net GPIO3: now also R28.1
- net GPIO4: now also R29.1
- net GPIO5: now also R30.1
- net RUN: now also SW1.2, SW1.4
- new net: L2.2 (A), R31.1
- new net: L1.2 (A), R32.1
- no-connect marks 31 -> 29

Commit message: HW Rev. 1.0 (final)
Parts:
- J1: footprint Connector_PinHeader_2.54mm:PinHeader_1x02_P2.54mm_Vertical -> LIBS:Boot_Jumper
- renumbered L2 to L1, L1 to L2, R8 to R10, R9 to R11, R10 to R12, R11 to R13, R12 to R14, R13 to R15, R14 to R16, R15 to R17, R16 to R18, R27 to R19, R28 to R20, R29 to R21, R30 to R22, R17 to R23, R18 to R24, R19 to R25, R20 to R26, R21 to R27, R22 to R28, R23 to R29, R24 to R30, R25 to R31, R26 to R32, R31 to R7, R32 to R8, R7 to R9
Other:
- company: Raspberry Pi Ltd -> Mikhail Matveev
- title: RP2040 Minimal Design Example -> Mini FRANK

Commit message: HW Rev 1.1
Parts:
- removed J1: Conn_01x02, LIBS:Boot_Jumper, symbol Connector_Generic:Conn_01x02
- added SW2: Flash Button, LIBS:Button_SMD_3x3x2, symbol Switch:SW_Push_Dual
- SW1: footprint LIBS:Button_SMD_6x6x5 -> LIBS:Button_SMD_3x3x2
Connections:
- net GND: now also SW2.1, SW2.3
- net ~{USB_BOOT}: now also SW2.2, SW2.4
Other:
- moved on the sheet: L2, R8

Commit message: HW Rev. 1.2
Parts:
- removed R3: DNF, Resistor_SMD:R_0805_2012Metric_Pad1.20x1.40mm_HandSolder, symbol Device:R
Connections:
- net GND: now also SW1.2, SW2.2; no longer SW1.3, SW2.3
- net RUN: now also SW1.3; no longer SW1.2
- net ~{USB_BOOT}: now also SW2.3; no longer SW2.2

Commit message: HW Rev 1.3
Parts:
- C1, C10, C11, C13, C14, C15, C16, C17, C18, C19, C2, C20, C23, C24, C3, C4, C5, C6, C7, C8, C9: footprint Capacitor_SMD:C_0805_2012Metric_Pad1.18x1.45mm_HandSolder -> LIBS:Medved_C_0805
- C21, C22: footprint LIBS:Medved_CP_Radial_D5.0mm_P2.50mm -> LIBS:Medved_C_0805
- D1, D2, D3: footprint LIBS:R_0805_PLUS -> LIBS:Medved_D_0805
- R1, R10, R11, R12, R13, R14, R15, R16, R17, R18, R19, R2, R20, R21, R22, R23, R24, R25, R26, R27, R28, R29, R30, R31, R32, R4, R5, R6, R7, R8, R9: footprint Resistor_SMD:R_0805_2012Metric_Pad1.20x1.40mm_HandSolder -> LIBS:Medved_R_0805

Commit message: HW Rev 1.4
Parts:
- added D4: 3V3, LIBS:Medved_D_0805, symbol Device:D_Zener
- added DB2: Joystick, Connector_Dsub:DSUB-9_Male_EdgeMount_P2.77mm, symbol Connector:DB9_Male
- added R3: 1k, LIBS:Medved_R_0805, symbol Device:R
Connections:
- net GND: now also D4.2 (A), DB2.8
- net GPIO14: now also DB2.4
- net GPIO15: now also DB2.3
- net GPIO17: now also D4.1 (K), R3.1
- net J1_DATA: now also DB2.2, R3.2
- net VBUS: now also DB2.6
- no-connect marks 29 -> 33
Other:
- added sheet PSRAM (psram.kicad_sch)
- note added: "Make sure R11 and R12 are close to RP2040"
- note removed: "Make sure R3 and R4 are close to RP2040"
- moved on the sheet: D1, DB1, R2

Commit message: Updates to HW Rev 1.4
Parts:
- C12: footprint Capacitor_SMD:C_0805_2012Metric_Pad1.18x1.45mm_HandSolder -> LIBS:Medved_C_0805
Changed lines of the file:
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@@
 			)
 		)
-		(property "Footprint" "Capacitor_SMD:C_0805_2012Metric_Pad1.18x1.45mm_HandSolder"
+		(property "Footprint" "LIBS:Medved_C_0805"
 			(at 224.4852 85.09 0)
 			(effects
