File: minifrank.kicad_sch (KiCad schematic)
At the start: 75 parts, among them SW1 Reset Button, SW2 Flash Button, U1 W25Q128JVS, U2 NCP1117-3.3_SOT223, U3 RP2040, Y1 ABM8-272-T3

Commit message: HW Rev 1.5
Parts:
- added C20: 10u, LIBS:Medved_CP_Radial_D5.0mm_P2.50mm, symbol Device:C_Polarized
- added JP1: Audio Jumpers, LIBS:Medved_JMP_2x03, symbol Connector_Generic:Conn_02x03_Odd_Even
- added JP2: I2S, LIBS:Medved_PinHeader_1x02, symbol Connector_Generic:Conn_01x02
- added TDA1: TDA1387T, Package_SO:SO-8_5.3x6.2mm_P1.27mm, symbol TDA1387T:TDA1387T
- renumbered C9 to C10, C20 to C21, C21 to C22, C22 to C23, C23 to C24, C24 to C25, C10 to C5, C5 to C6, C6 to C7, C7 to C8, C8 to C9, D4 to D2, D2 to D3, D3 to D4, R2 to R1, R13 to R11, R14 to R12, R11 to R13, R12 to R14, R3 to R2, R1 to R3, SW2 to SW1, SW1 to SW2
Connections:
- net GND: now also C20.2, TDA1.4 (AGND)
- net GPIO26: now also JP1.2 (Pin_2), TDA1.3 (DATA); no longer R32.2
- net GPIO27: now also JP1.4 (Pin_4), TDA1.1 (SCLK); no longer R29.2
- net GPIO28: now also JP1.6 (Pin_6), TDA1.2 (LRCK); no longer R30.2, R31.2
- net VBUS: now also TDA1.5 (VA)
- net L: no longer names the net of AU1.T, C22.2, R17.1
- net R: no longer names the net of AU1.R, C23.2, R18.1
- new net BEEP_OUT: JP1.5 (Pin_5), R30.2, R31.2
- new net FLT: C20.1, TDA1.7 (FLT)
- new net LEFT_OUT: JP1.3 (Pin_3), R29.2
- new net LEFT_TDA: JP2.2 (Pin_2), TDA1.6 (A_LEFT)
- new net RIGHT_OUT: JP1.1 (Pin_1), R32.2
- new net RIGHT_TDA: JP2.1 (Pin_1), TDA1.8 (A_RIGHT)
- no-connect marks 33 -> 28
Other:
- moved on the sheet: C5, D3, D4, KB1, R10, R11, R12, R9
