File: psram.kicad_sch (KiCad schematic)
At the start: 3 parts

Commit message: Updates to HW Rev 1.4
Parts:
- renumbered JP8 to JP1
Changed lines of the file:
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@@
 		(on_board yes)
 		(dnp no)
-		(property "Reference" "JP8"
+		(property "Reference" "JP1"
 			(at 91.44 64.77 0)
 			(effects

Commit message: HW Rev 1.4
Other:
- title: FRANK2 -> Mini FRANK
Changed lines of the file:
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@@
 	(generator "eeschema")
 	(generator_version "8.0")
-	(paper "A4")
+	(paper "A3")
 	(title_block
-		(title "FRANK2")
-		(date "2024-11-21")
-		(rev "1.0")
+		(title "Mini FRANK")
+		(date "2024-11-28")
+		(rev "1.4")
 		(company "Mikhail Matveev")
-		(comment 1 "https://github.com/xtremespb/frank2")
+		(comment 1 "https://github.com/xtremespb/minifrank")
 	)
 	(junction

Commit message: HW Rev 1.5
Parts:
- renumbered C30 to C26, JP1 to JP3
Changed lines of the file:
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@@
 		(title "Mini FRANK")
 		(date "2024-11-28")
-		(rev "1.4")
+		(rev "1.5")
 		(company "Mikhail Matveev")
 		(comment 1 "https://github.com/xtremespb/minifrank")
@@
 		(on_board yes)
 		(dnp no)
-		(property "Reference" "#PWR057"
+		(property "Reference" "#PWR047"
 			(at 62.23 72.39 0)
 			(effects
@@
 			(project "frank2"
 				(path "/8c0b3d8b-46d3-4173-ab1e-a61765f77d61/447aa656-0f67-4c4e-9e1e-c2d42aca6373"
-					(reference "#PWR057")
+					(reference "#PWR047")
 					(unit 1)
 				)
@@
 		(dnp no)
 		(fields_autoplaced yes)
-		(property "Reference" "#PWR043"
+		(property "Reference" "#PWR048"
 			(at 68.58 40.64 0)
 			(effects
@@
 			(project ""
 				(path "/8c0b3d8b-46d3-4173-ab1e-a61765f77d61/447aa656-0f67-4c4e-9e1e-c2d42aca6373"
-					(reference "#PWR043")
+					(reference "#PWR048")
 					(unit 1)
 				)
@@
 		(on_board yes)
 		(dnp no)
-		(property "Reference" "C30"
+		(property "Reference" "C26"
 			(at 44.831 47.0916 0)
 			(effects
@@
 			(project "frank2"
 				(path "/8c0b3d8b-46d3-4173-ab1e-a61765f77d61/447aa656-0f67-4c4e-9e1e-c2d42aca6373"
-					(reference "C30")
+					(reference "C26")
 					(unit 1)
 				)
@@
 		(on_board yes)
 		(dnp no)
-		(property "Reference" "JP1"
+		(property "Reference" "JP3"
 			(at 91.44 64.77 0)
 			(effects
@@
 			(project "frank2"
 				(path "/8c0b3d8b-46d3-4173-ab1e-a61765f77d61/447aa656-0f67-4c4e-9e1e-c2d42aca6373"
-					(reference "JP1")
+					(reference "JP3")
 					(unit 1)
 				)
@@
 		(on_board yes)
 		(dnp no)
-		(property "Reference" "#PWR056"
+		(property "Reference" "#PWR046"
 			(at 41.91 62.23 0)
 			(effects
@@
 			(project "frank2"
 				(path "/8c0b3d8b-46d3-4173-ab1e-a61765f77d61/447aa656-0f67-4c4e-9e1e-c2d42aca6373"
-					(reference "#PWR056")
+					(reference "#PWR046")
 					(unit 1)
 				)
